File: bread_board.brd (EAGLE design)
At the start: 40 x 50 mm, 7 parts, among them J2 DC_JACK

Commit message: Straightened up the lines and added text
Routing:
- net N$7: track 39.9 -> 45.1 mm
- net N$8: track 30.2 -> 34.9 mm
- net N$9: track 22.0 -> 25.3 mm
- net N$4: track 53.4 -> 55.3 mm
Other:
- board text added: "AUDIO-AMP"
Changed lines of the file:
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@@
 <?xml version="1.0" encoding="utf-8"?>
 <!DOCTYPE eagle SYSTEM "eagle.dtd">
-<eagle version="8.3.2">
+<eagle version="7.7.0">
 <drawing>
 <settings>
@@
 <text x="6" y="0.25" size="1.778" layer="21">GND</text>
 <text x="6" y="48" size="1.778" layer="21">9V+</text>
+<text x="32" y="11" size="1.778" layer="16" rot="MR0">AUDIO-AMP</text>
 </plain>
 <attributes>
@@
 </autorouter>
 <elements>
-<element name="SV1" library="con-lstb" library_urn="urn:adsk.eagle:library:162" package="MA04-1" package3d_urn="urn:adsk.eagle:package:8337/1" value="" x="3" y="4">
+<element name="SV1" library="con-lstb" package="MA04-1" value="" x="3" y="4">
 <attribute name="MF" value="" x="3" y="4" size="1.778" layer="27" display="off"/>
 <attribute name="MPN" value="" x="3" y="4" size="1.778" layer="27" display="off"/>
@@
 <attribute name="OC_NEWARK" value="unknown" x="3" y="4" size="1.778" layer="27" display="off"/>
 </element>
-<element name="SV2" library="con-lstb" library_urn="urn:adsk.eagle:library:162" package="MA04-1" package3d_urn="urn:adsk.eagle:package:8337/1" value="" x="3" y="11">
+<element name="SV2" library="con-lstb" package="MA04-1" value="" x="3" y="11">
 <attribute name="MF" value="" x="3" y="11" size="1.778" layer="27" display="off"/>
 <attribute name="MPN" value="" x="3" y="11" size="1.778" layer="27" display="off"/>
@@
 <attribute name="OC_NEWARK" value="unknown" x="3" y="11" size="1.778" layer="27" display="off"/>
 </element>
-<element name="SV3" library="con-lstb" library_urn="urn:adsk.eagle:library:162" package="MA04-1" package3d_urn="urn:adsk.eagle:package:8337/1" value="" x="3" y="46">
+<element name="SV3" library="con-lstb" package="MA04-1" value="" x="3" y="46">
 <attribute name="MF" value="" x="3" y="46" size="1.778" layer="27" display="off"/>
 <attribute name="MPN" value="" x="3" y="46" size="1.778" layer="27" display="off"/>
@@
 <attribute name="OC_NEWARK" value="unknown" x="3" y="46" size="1.778" layer="27" display="off"/>
 </element>
-<element name="SV4" library="con-lstb" library_urn="urn:adsk.eagle:library:162" package="MA04-1" package3d_urn="urn:adsk.eagle:package:8337/1" value="" x="3" y="39">
+<element name="SV4" library="con-lstb" package="MA04-1" value="" x="3" y="39">
 <attribute name="MF" value="" x="3" y="39" size="1.778" layer="27" display="off"/>
 <attribute name="MPN" value="" x="3" y="39" size="1.778" layer="27" display="off"/>
@@
 <wire x1="13.662825" y1="36.6002" x2="14.6002" y2="35.662825" width="1.016" layer="1"/>
 <wire x1="-2.6002" y1="36.6002" x2="13.662825" y2="36.6002" width="1.016" layer="1"/>
-<wire x1="14.6002" y1="35.662825" x2="14.6002" y2="32" width="1.016" layer="1"/>
-<wire x1="14.6002" y1="32" x2="14.6002" y2="31.5498" width="1.016" layer="1"/>
-<wire x1="14.6002" y1="32" x2="14.6002" y2="31.3998" width="1.016" layer="1"/>
-<wire x1="14.6002" y1="31.3998" x2="21" y2="25" width="1.016" layer="1"/>
-<wire x1="21" y1="25" x2="23.9" y2="25" width="1.016" layer="1"/>
 <wire x1="23.9" y1="25" x2="24.15" y2="24.75" width="1.016" layer="1"/>
+<wire x1="14.6002" y1="35.662825" x2="14.6002" y2="27.3998" width="1.016" layer="1"/>
+<wire x1="14.6002" y1="27.3998" x2="17" y2="25" width="1.016" layer="1"/>
+<wire x1="17" y1="25" x2="23.9" y2="25" width="1.016" layer="1"/>
 </signal>
 <signal name="N$5">
@@
 <wire x1="-0.81" y1="39" x2="-0.81" y2="41.19" width="0.8128" layer="1"/>
 <wire x1="-0.81" y1="41.19" x2="1.9172" y2="43.9172" width="0.8128" layer="1"/>
-<wire x1="1.9172" y1="43.9172" x2="19.0828" y2="43.9172" width="0.8128" layer="1"/>
-<wire x1="19.0828" y1="43.9172" x2="30.5" y2="32.5" width="0.8128" layer="1"/>
-<wire x1="30.5" y1="32.5" x2="30.5" y2="32" width="0.8128" layer="1"/>
+<wire x1="1.9172" y1="43.9172" x2="28.0828" y2="43.9172" width="0.8128" layer="1"/>
+<wire x1="28.0828" y1="43.9172" x2="30.5" y2="41.5" width="0.8128" layer="1"/>
+<wire x1="30.5" y1="41.5" x2="30.5" y2="32" width="0.8128" layer="1"/>
 </signal>
 <signal name="N$8">
@@
 <wire x1="1.73" y1="39" x2="1.73" y2="40.73" width="0.8128" layer="1"/>
 <wire x1="1.73" y1="40.73" x2="3.952" y2="42.952" width="0.8128" layer="1"/>
-<wire x1="3.952" y1="42.952" x2="14.048" y2="42.952" width="0.8128" layer="1"/>
-<wire x1="14.048" y1="42.952" x2="24.5" y2="32.5" width="0.8128" layer="1"/>
-<wire x1="24.5" y1="32.5" x2="24.5" y2="32" width="0.8128" layer="1"/>
+<wire x1="3.952" y1="42.952" x2="22.048" y2="42.952" width="0.8128" layer="1"/>
+<wire x1="22.048" y1="42.952" x2="24.5" y2="40.5" width="0.8128" layer="1"/>
+<wire x1="24.5" y1="40.5" x2="24.5" y2="32" width="0.8128" layer="1"/>
 </signal>
 <signal name="N$9">
@@
 <wire x1="4.27" y1="39" x2="4.27" y2="40.27" width="0.8128" layer="1"/>
 <wire x1="4.27" y1="40.27" x2="5.9868" y2="41.9868" width="0.8128" layer="1"/>
-<wire x1="5.9868" y1="41.9868" x2="11.2632" y2="41.9868" width="0.8128" layer="1"/>
-<wire x1="11.2632" y1="41.9868" x2="18.5" y2="34.75" width="0.8128" layer="1"/>
-<wire x1="18.5" y1="34.75" x2="18.5" y2="32" width="0.8128" layer="1"/>
+<wire x1="5.9868" y1="41.9868" x2="17.0132" y2="41.9868" width="0.8128" layer="1"/>
+<wire x1="17.0132" y1="41.9868" x2="18.5" y2="40.5" width="0.8128" layer="1"/>
+<wire x1="18.5" y1="40.5" x2="18.5" y2="32" width="0.8128" layer="1"/>
 </signal>
 <signal name="N$2">
@@
 </board>
 </drawing>
-<compatibility>
-<note version="8.2" severity="warning">
-Since Version 8.2, EAGLE supports online libraries. The ids
-of those online libraries will not be understood (or retained)
-with this version.
-</note>
-<note version="8.3" severity="warning">
-Since Version 8.3, EAGLE supports URNs for individual library
-assets (packages, symbols, and devices). The URNs of those assets
-will not be understood (or retained) with this version.
-</note>
-<note version="8.3" severity="warning">
-Since Version 8.3, EAGLE supports the association of 3D packages
-with devices in libraries, schematics, and board files. Those 3D
-packages will not be understood (or retained) with this version.
-</note>
-</compatibility>
 </eagle>
